File: RTnexen_UPS_PMC.kicad_pcb (KiCad board)
At the start: 2 copper layers, 50 x 70 mm, 35 parts, among them J1 USB_A, J2 KF301-2P, U1 MP2393GTL-P, U2 INA226AIDGSR

Commit message: Update PCB layout
Parts:
- moved J1 56.0 mm to (245.5, 70.8)
- moved A1 56.0 mm to (215.7, 59.0)
- moved H1 56.0 mm to (214.3, 53.5)
- moved H2 56.0 mm to (254.3, 53.5)
- moved H3 56.0 mm to (214.3, 113.5)
- moved H4 56.0 mm to (254.3, 113.5)
- moved J2 56.0 mm to (241.6, 113.2)
- moved 50mR1 40.2 mm to (100.1, 89.2), turned to 90 degrees
- moved C9 28.4 mm to (99.5, 80.4), turned to -90 degrees
- moved U2 24.2 mm to (93.2, 88.7)
- moved R9 23.5 mm to (88.0, 88.2)
- moved R10 23.0 mm to (88.0, 89.2)
- moved R11 22.5 mm to (88.0, 90.2)
Routing:
- net +3.3V: track 0.00 -> 10.6 mm
- net /ALERT_INA226: track 0.00 -> 2.67 mm, vias 0 -> 1
- net /SCL_INA226: track 0.00 -> 2.67 mm, vias 0 -> 1
- net /SDA_INA226: track 0.00 -> 2.46 mm, vias 0 -> 1

Commit message: Update PCB layout
Parts:
- moved C11 199.3 mm to (252.5, 162.3), turned to -90 degrees
- moved C10 196.7 mm to (251.7, 155.7), turned to 90 degrees
- moved 50mR1 176.0 mm to (261.6, 159.3)
- moved R10 172.2 mm to (245.3, 159.5)
- moved R11 172.2 mm to (245.3, 160.5)
- moved R9 172.2 mm to (245.3, 158.5)
- moved U2 172.2 mm to (250.4, 159.0)
- moved C9 170.8 mm to (252.7, 155.7), turned to 90 degrees
- moved R1 32.5 mm to (75.4, 80.5)
- moved C1 30.8 mm to (72.4, 78.2), turned to 180 degrees
- moved C2 29.9 mm to (72.4, 79.2), turned to 180 degrees
- moved R3 27.4 mm to (78.2, 79.2), turned to 180 degrees
- moved C4 26.6 mm to (79.3, 80.5)
- moved C3 26.3 mm to (78.2, 78.2), turned to 180 degrees
- moved R6 19.5 mm to (72.4, 77.2), turned to 180 degrees
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Routing:
- net /Power/VIN: track 0.00 -> 5.40 mm
- net Net-(U2-IN-): track 0.00 -> 3.27 mm
- net /PG_MP2393: track 0.00 -> 3.04 mm
- net /EN_MP2393: track 0.00 -> 2.43 mm
- net Net-(U2-IN+): track 0.00 -> 1.88 mm
- net +3.3V: track 10.6 -> 12.5 mm
- net Net-(U1-SS): track 0.00 -> 1.53 mm
- net Net-(U1-BST): track 0.00 -> 1.53 mm
- net Net-(C4-Pad1): track 0.00 -> 1.29 mm
